File: _autosave-horizon-mini.kicad_sch (KiCad schematic)
At the start: 75 parts, among them J2 Conn_01x02_Pin, J3 Micro_SD_Card_Det1, J7 USB_C_Receptacle_USB2.0_16P, J8 Conn_02x03_Counter_Clockwise, Q1 BSS138, Q10 DMG2301L, U1 TPS82130, U16 AP2112K-3.3, U2 TPS61092, U3 LTC4412xS6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

Commit message: Deleted unneeded chips and changes sensors from spi to i2c
Parts:
- removed R26: R, Resistor_SMD:R_0603_1608Metric, symbol Device:R
- U4: value TMCU -> MCU
Connections:
- net CS_IMU TMCU: no longer names the net of U4.32 (PA15)
- net INTERRUPT TMCU: no longer names the net of R28.2, U9.4 (INT1)
Other:
- moved on the sheet: R28
Changed lines of the file:
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@@
 	)
 	(junction
-		(at 50.8 140.97)
-		(diameter 0)
-		(color 0 0 0 0)
-	)
-	(junction
 		(at -53.34 102.87)
 		(diameter 0)
@@
 	(wire
 		(pts
-			(xy -27.94 54.61) (xy -31.75 54.61)
-		)
-		(stroke
-			(width 0)
-			(type default)
-		)
-	)
-	(wire
-		(pts
 			(xy 231.14 157.48) (xy 231.14 154.94)
 		)
@@
 	(wire
 		(pts
-			(xy 49.53 140.97) (xy 50.8 140.97)
+			(xy 252.73 40.64) (xy 252.73 55.88)
 		)
 		(stroke
@@
 	(wire
 		(pts
-			(xy 252.73 40.64) (xy 252.73 55.88)
+			(xy 90.17 95.25) (xy 92.71 95.25)
 		)
 		(stroke
@@
 	(wire
 		(pts
-			(xy 90.17 95.25) (xy 92.71 95.25)
+			(xy -31.75 54.61) (xy -29.21 54.61)
 		)
 		(stroke
@@
 	(wire
 		(pts
-			(xy 50.8 140.97) (xy 69.85 140.97)
-		)
-		(stroke
-			(width 0)
-			(type default)
-		)
-	)
-	(wire
-		(pts
 			(xy 238.76 129.54) (xy 238.76 132.08)
 		)
@@
 		)
 	)
-	(global_label "INTERRUPT TMCU"
-		(shape input)
-		(at -27.94 54.61 0)
-		(fields_autoplaced yes)
-		(effects
-			(font
-				(size 1.27 1.27)
-			)
-			(justify left)
-		)
-		(property "Intersheetrefs" "${INTERSHEET_REFS}"
-			(at -8.8077 54.61 0)
-			(effects
-				(font
-					(size 1.27 1.27)
-				)
-				(justify left)
-				(hide yes)
-			)
-		)
-	)
 	(global_label "MISO TMCU"
 		(shape input)
@@
 		)
 	)
-	(global_label "CS_IMU TMCU"
-		(shape input)
-		(at 49.53 140.97 180)
-		(fields_autoplaced yes)
-		(effects
-			(font
-				(size 1.27 1.27)
-			)
-			(justify right)
-		)
-		(property "Intersheetrefs" "${INTERSHEET_REFS}"
-			(at 33.7239 140.97 0)
-			(effects
-				(font
-					(size 1.27 1.27)
-				)
-				(justify right)
-				(hide yes)
-			)
-		)
-	)
 	(global_label "2B"
 		(shape input)
@@
 		(on_board yes)
 		(dnp no)
-		(fields_autoplaced yes)
 		(property "Reference" "#PWR061"
 			(at -30.48 46.99 0)
@@
 		)
 		(property "Value" "GND"
-			(at -33.02 46.9899 90)
+			(at -21.5899 49.53 0)
 			(effects
 				(font
@@
 	(symbol
 		(lib_id "power:+3.3V")
-		(at -27.94 46.99 0)
+		(at -21.59 54.61 270)
 		(unit 1)
 		(exclude_from_sim no)
@@
 		(dnp no)
 		(property "Reference" "#PWR071"
-			(at -27.94 50.8 0)
+			(at -25.4 54.61 0)
 			(effects
 				(font
@@
 		)
 		(property "Value" "+3.3V"
-			(at -27.94 41.656 90)
+			(at -16.256 54.61 90)
 			(effects
 				(font
@@
 		)
 		(property "Footprint" ""
-			(at -27.94 46.99 0)
+			(at -21.59 54.61 0)
 			(effects
 				(font
@@
 		)
 		(property "Datasheet" ""
-			(at -27.94 46.99 0)
+			(at -21.59 54.61 0)
 			(effects
 				(font
@@
 		)
 		(property "Description" "Power symbol creates a global label with name \"+3.3V\""
-			(at -27.94 46.99 0)
+			(at -21.59 54.61 0)
 			(effects
 				(font
@@
 	)
 	(symbol
-		(lib_id "power:+3.3V")
-		(at 50.8 148.59 180)
-		(unit 1)
-		(exclude_from_sim no)
-		(in_bom yes)
-		(on_board yes)
-		(dnp no)
-		(property "Reference" "#PWR095"
-			(at 50.8 144.78 0)
-			(effects
-				(font
-					(size 1.27 1.27)
-				)
-				(hide yes)
-			)
-		)
-		(property "Value" "+3.3V"
-			(at 50.8 153.924 90)
-			(effects
-				(font
-					(size 1.27 1.27)
-				)
-			)
-		)
-		(property "Footprint" ""
-			(at 50.8 148.59 0)
-			(effects
-				(font
-					(size 1.27 1.27)
-				)
-				(hide yes)
-			)
-		)
-		(property "Datasheet" ""
-			(at 50.8 148.59 0)
-			(effects
-				(font
-					(size 1.27 1.27)
-				)
-				(hide yes)
-			)
-		)
-		(property "Description" "Power symbol creates a global label with name \"+3.3V\""
-			(at 50.8 148.59 0)
-			(effects
-				(font
-					(size 1.27 1.27)
-				)
-				(hide yes)
-			)
-		)
-		(pin "1"
-		)
-		(instances
-			(project "horizon-mini"
-				(path "/2e9ea5c6-e973-4316-a82c-e40ce72f6995"
-					(reference "#PWR095")
-					(unit 1)
-				)
-			)
-		)
-	)
-	(symbol
 		(lib_id "Device:R")
 		(at 129.54 173.99 90)
@@
 			)
 		)
-		(property "Value" "TMCU"
+		(property "Value" "MCU"
 			(at 85.852 153.416 0)
 			(effects
@@
 	)
 	(symbol
-		(lib_id "Device:R")
-		(at 50.8 144.78 0)
-		(unit 1)
-		(exclude_from_sim no)
-		(in_bom yes)
-		(on_board yes)
-		(dnp no)
-		(property "Reference" "R26"
-			(at 45.466 145.034 0)
-			(effects
-				(font
-					(size 1.27 1.27)
-				)
-				(justify left)
-			)
-		)
-		(property "Value" "R"
-			(at 45.466 147.574 0)
-			(effects
-				(font
-					(size 1.27 1.27)
-				)
-				(justify left)
-			)
-		)
-		(property "Footprint" "Resistor_SMD:R_0603_1608Metric"
-			(at 49.022 144.78 90)
-			(effects
-				(font
-					(size 1.27 1.27)
-				)
-				(hide yes)
-			)
-		)
-		(property "Datasheet" "~"
-			(at 50.8 144.78 0)
-			(effects
-				(font
-					(size 1.27 1.27)
-				)
-				(hide yes)
-			)
-		)
-		(property "Description" "Resistor"
-			(at 50.8 144.78 0)
-			(effects
-				(font
-					(size 1.27 1.27)
-				)
-				(hide yes)
-			)
-		)
-		(pin "2"
-		)
-		(pin "1"
-		)
-		(instances
-			(project "horizon-mini"
-				(path "/2e9ea5c6-e973-4316-a82c-e40ce72f6995"
-					(reference "R26")
-					(unit 1)
-				)
-			)
-		)
-	)
-	(symbol
 		(lib_id "power:GND")
 		(at -55.88 165.1 270)
@@
 		)
 		(property "Value" "SMLVN6RGB"
-			(at -96.52 137.16 0)
+			(at -96.52 115.57 0)
 			(effects
 				(font
@@
 	(symbol
 		(lib_id "Device:R")
-		(at -27.94 50.8 0)
+		(at -25.4 54.61 270)
 		(unit 1)
 		(exclude_from_sim no)
@@
 		(fields_autoplaced yes)
 		(property "Reference" "R28"
-			(at -25.4 49.5299 0)
+			(at -24.1299 57.15 0)
 			(effects
 				(font
@@
 		)
 		(property "Value" "10k"
-			(at -25.4 52.0699 0)
+			(at -26.6699 57.15 0)
 			(effects
 				(font
@@
 		)
 		(property "Footprint" "Resistor_SMD:R_0603_1608Metric"
-			(at -29.718 50.8 90)
+			(at -25.4 52.832 90)
 			(effects
 				(font
@@
 		)
 		(property "Datasheet" "~"
-			(at -27.94 50.8 0)
+			(at -25.4 54.61 0)
 			(effects
 				(font
@@
 		)
 		(property "Description" "Resistor"
-			(at -27.94 50.8 0)
+			(at -25.4 54.61 0)
 			(effects
 				(font
