File: horizon.kicad_sch (KiCad schematic)
At the start: 36 parts, among them J2 Conn_02x03_Counter_Clockwise, J7 Conn_02x03_Counter_Clockwise, J8 Conn_02x03_Counter_Clockwise, U1 MMCU, U3 NMCU, U4 TMCU, Y1 Crystal

Commit message: Deleted unneeded chips and changes sensors from spi to i2c
Parts:
- removed C63, C72: 1uF, Capacitor_SMD:C_0603_1608Metric, symbol Device:C
- removed C64, C65, C66: 0.1uF, Capacitor_SMD:C_0603_1608Metric, symbol Device:C
- removed C67: 4.7uF, Capacitor_SMD:C_0603_1608Metric, symbol Device:C
- removed C73, C74, C75, C76, C77, C79: 100nF, Capacitor_SMD:C_0603_1608Metric, symbol Device:C
- removed J2, J7: Conn_02x03_Counter_Clockwise, Connector_PinHeader_2.54mm:PinHeader_2x03_P2.54mm_Vertical, symbol Connector_Generic:Conn_02x03_Counter_Clockwise
- removed R30: R, Resistor_SMD:R_0603_1608Metric, symbol Device:R
- removed U1: MMCU, MK20DX256VLH7:QFP50P1200X1200X160-64N, symbol MK20DX256VLH7:MK20DX256VLH7
- removed U3: NMCU, Package_QFP:TQFP-64_10x10mm_P0.5mm, symbol MCU_Microchip_SAMD:ATSAMD21J16B-A
- removed Y1: Crystal, Crystal:Crystal_AT310_D3.0mm_L10.0mm_Vertical, symbol Device:Crystal
- added BZ2: Buzzer, Buzzer_Beeper:MagneticBuzzer_PUI_AT-0927-TT-6-R, symbol Device:Buzzer
- added C1, C2, C3, C4, C5: 100nF, Capacitor_SMD:C_0603_1608Metric, symbol Device:C
- added C14: 3.3 nF, Capacitor_SMD:C_0603_1608Metric, symbol Device:C
- added C28: 4n7, Capacitor_SMD:C_0603_1608Metric, symbol Device:C
- added C29: 100n, Capacitor_SMD:C_0603_1608Metric, symbol Device:C
- added C37: 22uF, Capacitor_SMD:C_0603_1608Metric, symbol Device:C
- added C38: 1uF, Capacitor_SMD:C_0603_1608Metric, symbol Device:C
- added C39: 2u2, Capacitor_SMD:C_0603_1608Metric, symbol Device:C
- added C40: 10uF, Capacitor_SMD:C_0603_1608Metric, symbol Device:C
- added C46: 100u, Capacitor_SMD:C_0603_1608Metric, symbol Device:C_Polarized_US
- added C47: 1u, Capacitor_SMD:C_0603_1608Metric, symbol Device:C
- added D1: SMLVN6RGB, LED_SMD:LED_ROHM_SMLVN6, symbol LED:SMLVN6RGB
- added D10, D13, D5, D6: PMEG6020ER, Diode_SMD:Nexperia_CFP3_SOD-123W, symbol Diode:PMEG6020ER
- added D11, D12, D9: LED, LED_SMD:LED_0603_1608Metric, symbol Device:LED
- added D14: PRTR5V0U2X, Package_TO_SOT_SMD:SOT-143, symbol Power_Protection:PRTR5V0U2X
- added J2: Conn_01x02_Pin, Connector_JST:JST_PH_B2B-PH-K_1x02_P2.00mm_Vertical, symbol Connector:Conn_01x02_Pin
- added J3: Micro_SD_Card_Det1, Connector_Card:microSD_HC_Hirose_DM3D-SF, symbol Connector:Micro_SD_Card_Det1
- added J7: USB_C_Receptacle_USB2.0_16P, Connector_USB:USB_C_Receptacle_GCT_USB4105-xx-A_16P_TopMnt_Horizontal, symbol Connector:USB_C_Receptacle_USB2.0_16P
- added L7: SLF7055T-6R8N2R8-3PF, Inductor_SMD:L_7.3x7.3_H4.5, symbol SLF7055T-6R8N2R8-3PF[1]:SLF7055T-6R8N2R8-3PF
- added Q1: BSS138, Package_TO_SOT_SMD:SOT-23, symbol Transistor_FET:BSS138
- added Q10: DMG2301L, Package_TO_SOT_SMD:SOT-23, symbol Transistor_FET:DMG2301L
- added R1: 2k2, Resistor_SMD:R_0603_1608Metric, symbol Device:R
- added R10: 100k, Resistor_SMD:R_0603_1608Metric, symbol Device:R
- added R11, R2, R23: 10kΩ, Resistor_SMD:R_0603_1608Metric, symbol Device:R
- added R13, R18, R19: 220, Resistor_SMD:R_0603_1608Metric, symbol Device:R
- added R14, R17: 330, Resistor_SMD:R_0603_1608Metric, symbol Device:R
- added R15, R16: 5k1, Resistor_SMD:R_0603_1608Metric, symbol Device:R
- added R21, R22, R25, R28: 10k, Resistor_SMD:R_0603_1608Metric, symbol Device:R
- added R8: 100, Resistor_SMD:R_0603_1608Metric, symbol Device:R
- added R9: 430k, Resistor_SMD:R_0603_1608Metric, symbol Device:R
- added TP1, TP2: TestPoint, TestPoint:TestPoint_Pad_1.0x1.0mm, symbol Connector:TestPoint
- added U1: TPS82130, Package_LGA:Texas_SIL0008D_MicroSiP-8-1EP_2.8x3mm_P0.65mm_EP1.1x1.9mm_ThermalVias, symbol Regulator_Switching:TPS82130
- added U16: AP2112K-3.3, Package_TO_SOT_SMD:SOT-23-5, symbol Regulator_Linear:AP2112K-3.3
- added U2: TPS61092, Package_DFN_QFN:Texas_RSA_VQFN-16-1EP_4x4mm_P0.65mm_EP2.7x2.7mm_ThermalVias, symbol Regulator_Switching:TPS61092
- added U3: LTC4412xS6, Package_TO_SOT_SMD:TSOT-23-6, symbol Power_Management:LTC4412xS6
- added U6: NAND, Package_SO:SOIC-8_5.3x5.3mm_P1.27mm, symbol Memory_Flash:W25Q128JVS
- added U7: LPS22HB, Package_LGA:ST_HLGA-10_2x2mm_P0.5mm_LayoutBorder3x2y, symbol Sensor_Pressure:LPS22HB
- added U9: LSM6DS3, Package_LGA:LGA-14_3x2.5mm_P0.5mm_LayoutBorder3x4y, symbol Sensor_Motion:LSM6DS3
- C10: value 12pF -> 10uF
- C17: value 12pF -> 10u
- R29: value R -> 10k
- R3, R4: value 10k -> 100k
- R6: value 4.7k -> 350k
- R7: value 4.7k -> 100k
Connections:
- net RF_CS is gone; now on net CS_NAND MMCU: U4.16 (PA07)
- net nRESET DMCU-1 is gone; now on an unnamed net: R3.1
- net sda is gone; now on net GND: R7.2
- net +3.3V: now also R29.1, BZ2.1 (+), C1.1, C2.2, C3.2, C4.2, C47.1, C5.2, J3.4 (VDD), R11.1, R14.1, R2.1, R21.1, R22.1, R23.1, R25.1, R28.1, U16.5 (VOUT), U6.8 (VCC), U7.1 (Vdd_IO), U7.10 (VDD), U9.5 (VDDIO), U9.8 (VDD); no longer R29.2, R3.2, R4.2, R6.1, R7.1
- net 2B: now also R19.1
- net 2G: now also R18.1
- net 2R: now also R13.1
- net BUZZER: now also U4.17 (PA08), Q1.1 (G), R1.1
- net CS_NAND MMCU: now also U6.1 (~{CS})
- net CS_SD MMCU: now also U4.24 (PB11), J3.2 (DAT3/CD), R23.2; no longer R29.1
- net D+ DMCU-2: now also D14.2 (I/O1), J7.A6 (D+), J7.B6 (D+), TP1.1
- net D- DMCU-2: now also D14.3 (I/O2), J7.A7 (D-), J7.B7 (D-), TP2.1
- net GND: now also R4.2, C1.2, C14.2, C2.1, C28.1, C29.1, C3.1, C37.2, C38.2, C39.2, C4.1, C40.2, C46.2, C47.2, C5.1, D1.4 (GK), D1.5 (RK), D1.6 (BK), D11.1 (K), D12.1 (K), D14.1 (GND), D9.1 (K), J2.2 (Pin_2), J3.10 (SHIELD), J3.6 (VSS), J7.A1 (GND), J7.A12 (GND), J7.B1 (GND), J7.B12 (GND), J7.S1 (SHIELD), Q1.2 (S), R1.2, R10.2, R15.2, R16.2, U1.3 (GND), U1.9 (GND), U16.2 (GND), U2.10 (SYNC), U2.13 (GND), U2.17 (PAD), U2.5 (PGND), U2.6 (PGND), U2.7 (PGND), U3.2 (GND), U3.3 (CTL), U6.4 (GND), U7.3 (GND), U7.5 (SA0), U7.8 (GND), U7.9 (GND), U9.1 (SDO/SA0), U9.2 (SDX), U9.3 (SCX), U9.6 (GND), U9.7 (GND)
- net I2C0_SCL: now also U7.2 (SCL), U9.13 (SCL)
- net I2C0_SDA: now also U7.4 (SDA), U9.14 (SDA)
- net INTERRUPT TMCU: now also R28.2, U9.4 (INT1); no longer U4.31 (PA14)
- net MISO TMCU: now also J3.7 (DAT0), U6.2 (DO/IO_{1})
- net MOSI TMCU: now also J3.3 (CMD), U6.5 (DI/IO_{0})
- net SCK TMCU: now also J3.5 (CLK), U6.6 (CLK)
- net at C10.1: now also D6.1 (K), U1.1 (EN), U1.2 (VIN)
- net at C17.1: now also J2.1 (Pin_1), L7.1, U2.11 (EN), U2.8 (VBAT)
- net SD_DETECT: now reaches U4.23 (PB10)
- net SD_DETECT: now also J3.9 (DET), R22.2
- net CS_BARO TMCU: no longer names the net of U4.63 (PB02)
- net RX TMCU: no longer names the net of U4.14 (PA05)
- net TX TMCU: no longer names the net of U4.13 (PA04)
- net nRESET MMCU: no longer names the net of R4.1
- net nRESET MMCU: now also R3.2, U2.9 (LBI)
- net scl: no longer names the net of R6.2
- net scl: now also R7.1, U1.6 (FB)
- new net: D9.2 (A), R8.2
- new net: R25.2, U7.7 (INT_DRDY)
- new net: C37.1, C38.1, R6.1, R8.1, U1.4 (VOUT), U1.5 (VOUT), U16.1 (VIN), U16.3 (EN)
- new net: Q10.1 (G), U3.5 (GATE)
- new net: C28.2, C29.2, D13.2 (A), D14.4 (VCC), J7.A4 (VBUS), J7.A9 (VBUS), J7.B4 (VBUS), J7.B9 (VBUS), R17.2
- new net: R2.2, U6.7 (~{HOLD}/~{RESET}/IO_{3})
- new net: C14.1, U1.8 (SS/TR)
- new net: D1.1 (BA), R19.2
- new net: R11.2, U6.3 (~{WP}/IO_{2})
- new net: D12.2 (A), R17.1
- new net: D11.2 (A), R14.2
- new net: J7.A5 (CC1), R15.1
- new net: R21.2, U9.12 (CS)
- new net: R29.2, U7.6 (~{CS})
- new net: BZ2.2 (-), Q1.3 (D)
- new net: D1.3 (GA), R13.2
- new net: D1.2 (RA), R18.2
- new net: J7.B5 (CC2), R16.1
- new net: L7.2, U2.3 (SW), U2.4 (SW)
- new net: R10.1, R9.2, U2.14 (FB)
- new net +5V: D5.1 (K), D6.2 (A)
- new net POWAAAA: C40.1, D10.1 (K), D5.2 (A), Q10.2 (S), U3.6 (SENSE)
- new net VBUS: D10.2 (A), D13.1 (K)
- new net bat: C39.1, C46.1, Q10.3 (D), R9.1, U2.1 (VOUT), U2.15 (VOUT), U2.16 (VOUT), U3.1 (VIN)
- no-connect marks 78 -> 36
Other:
- removed sheet input usb
- removed sheet power stuff
- removed sheet sensors
- note added: "Baro"
- note added: "Storage/Logging"
- note removed: "Clock pin For NAND and SD"
- note removed: "For NAND and SD"
- note removed: "GPS → MCU RX"
- note removed: "INT from NAV"
- note removed: "INT from TLM"
- note removed: "MCU → GPS TX"
- note removed: "MISO"
- note removed: "MOSI"
- note removed: "Outputs a signal when data is ready"
- note removed: "Pull low to talk"
- note removed: "SERCOM Stuff For Firmware INTCOMM"
- moved on the sheet: C61, C62, C68, C69, C70, C71, C78, J8, R26, R5, U4
