File: horizon-mini.kicad_pcb (KiCad board)
At the start: 2 copper layers, 35 x 75 mm, 75 parts, among them J2 Conn_01x02_Pin, J3 Micro_SD_Card_Det1, J7 USB_C_Receptacle_USB2.0_16P, J8 Conn_02x03_Counter_Clockwise, Q1 BSS138, Q10 DMG2301L, U1 TPS82130, U16 AP2112K-3.3, U2 TPS61092, U3 LTC4412xS6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

Commit message: finish v2 traces
Routing:
- net +3.3V: track 109.0 -> 197.7 mm, vias 5 -> 9
- net GND: track 1.78 -> 63.1 mm, vias 0 -> 10
- net D+ DMCU-2: track 67.4 -> 82.4 mm
- net bat: track 14.9 -> 27.4 mm, vias 0 -> 2
- net D- DMCU-2: track 57.9 -> 68.1 mm
Other:
- board size 35 x 75 mm -> 35 x 60.5 mm
