File: Hardware/_autosave-horizon.kicad_sch (KiCad schematic)
At the start: 75 parts, among them J2 Conn_01x02_Pin, J3 Micro_SD_Card_Det1, J7 USB_C_Receptacle_USB2.0_16P, J8 Conn_02x03_Counter_Clockwise, Q1 BSS138, Q10 DMG2301L, U1 TPS82130, U16 AP2112K-3.3, U2 TPS61092, U3 LTC4412xS6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

Commit message: Deleted unneeded chips and changes sensors from spi to i2c
Connections:
- net CS_IMU TMCU: now also R21.2, U9.12 (CS)
- net CS_NAND MMCU: no longer U4.16 (PA07)
- net CS_SD MMCU: no longer U4.24 (PB11)
- net I2C0_SCL: no longer U9.13 (SCL)
- net I2C0_SDA: no longer U9.14 (SDA)
- new net RF_CS: U4.16 (PA07)
- no-connect marks 36 -> 39
Other:
- moved on the sheet: BZ2, C1, C10, C14, C17, C2, C28, C29, C3, C37, C38, C39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
