File: Hardware/horizon-mini.kicad_sch (KiCad schematic)
At the start: 76 parts, among them J2 Conn_01x02_Pin, J3 Micro_SD_Card_Det1, J7 USB_C_Receptacle_USB2.0_16P, J8 Conn_02x03_Counter_Clockwise, Q1 BSS138, Q10 DMG2301L, U1 TPS82130, U16 AP2112K-3.3, U2 TPS61092, U3 LTC4412xS6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

Commit message: Revert "Merge branch 'main' of https://github.com/Horizon-Avionics/Horizon-Mini"
This reverts commit 679f00b043b1fbfec2143f9512c96a76483b1c63, reversing
changes made to 3d15d739e12ed0ad8f757afd069957ffb8171449.
Parts:
- added C11: 0.1uF, Capacitor_SMD:C_0603_1608Metric, symbol Device:C
- C12: value 0.1uF -> 10uF
- C6: value 1uF -> F1uF
Connections:
- net +3.3V: no longer C7.1, C8.1, C9.1
- net GND: no longer C7.2, C8.2, C9.2, U5.17 (VDDIO), U5.36 (VDDIO), U5.44 (VDDIN)
- net at C12.1, U5.6 (VDDANA): now also C11.2
- new net: C8.2, U5.36 (VDDIO)
- new net: C9.2, U5.17 (VDDIO)
- new net: C7.2, U5.44 (VDDIN)

Commit message: fixed schematic
i hate github
Connections:
- net +3.3V: now also C11.2, C12.1, C7.2, C8.2, C9.1, U5.17 (VDDIO), U5.36 (VDDIO), U5.44 (VDDIN), U5.6 (VDDANA)
- net GND: now also C11.1, C12.2, C7.1, C8.1, C9.2
Other:
- moved on the sheet: C7, C8, C9
