File: Hardware/horizon-mini.kicad_pcb (KiCad board)
At the start: 2 copper layers, 34 x 34 mm, 77 parts, among them J2 Conn_01x02_Pin, J3 Micro_SD_Card_Det1, J7 USB_C_Receptacle_USB2.0_16P, J8 Conn_02x03_Counter_Clockwise, Q10 DMG2301L, U1 TPS82130, U16 AP2112K-3.3, U2 TPS61092, U3 LTC4412xS6, U5 ATSAMD21G18A-A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

Commit message: push
Parts:
- added BZ2: Buzzer, Buzzer_Beeper:MagneticBuzzer_PUI_AT-0927-TT-6-R, F.Cu at (117.0, 124.5)
- added D3: LED, LED_SMD:LED_0603_1608Metric, F.Cu at (110.5, 123.3)
- added D4: LED, LED_SMD:LED_0603_1608Metric, F.Cu at (107.9, 123.3)
- added F1: Polyfuse, Fuse:Fuse_0603_1608Metric, F.Cu at (121.0, 110.3)
- added F2: Polyfuse, Fuse:Fuse_0603_1608Metric, F.Cu at (118.5, 110.3)
- added J19: Screw_Terminal_01x02, TerminalBlock_Phoenix:TerminalBlock_Phoenix_MPT-0,5-2-2.54_1x02_P2.54mm_Horizontal, F.Cu at (131.8, 117.8)
- added J20: Screw_Terminal_01x02, TerminalBlock_Phoenix:TerminalBlock_Phoenix_MPT-0,5-2-2.54_1x02_P2.54mm_Horizontal, B.Cu at (139.6, 107.1)
- added Q1: BSS138, Package_TO_SOT_SMD:SOT-23, F.Cu at (119.9, 118.8)
- added Q8: IRLML6402, Package_TO_SOT_SMD:SOT-23, F.Cu at (115.3, 118.8)
- added Q9: IRLML6402, Package_TO_SOT_SMD:SOT-23, F.Cu at (110.7, 118.8)
- added R1: 2k2, Resistor_SMD:R_0603_1608Metric, F.Cu at (116.0, 110.3)
- added R58: 1k, Resistor_SMD:R_0603_1608Metric, F.Cu at (113.5, 110.3)
- added R59: 1k, Resistor_SMD:R_0603_1608Metric, F.Cu at (111.0, 110.3)
- added R79: 100, Resistor_SMD:R_0603_1608Metric, F.Cu at (121.0, 114.3)
- added R81: 100, Resistor_SMD:R_0603_1608Metric, F.Cu at (116.0, 114.3)
- C11: value 10uF -> 0.1uF
- C12: value 100nF -> 10uF
- C6: value 100nF -> F1uF
- C7, C8, C9: value 100nF -> 0.1uF
- J2: value Conn_01x02_Pin -> Screw_Terminal_01x02
- moved J8 10.9 mm to (144.2, 99.2), turned to 90 degrees
Connections:
- C11 pad 1: GND -> +3.3V
- C11 pad 2: +3.3V -> GND
- C6 pad 1: GND -> +3.3V
- C6 pad 2: Net-(U5-VDDCORE) -> GND
- C7 pad 1: GND -> +3.3V
- C7 pad 2: +3.3V -> GND
- C8 pad 1: GND -> +3.3V
- C8 pad 2: +3.3V -> GND
- C9 pad 1: GND -> +3.3V
- C9 pad 2: +3.3V -> GND
- D14 pad 2: D+ DMCU-2 -> Net-(D14-I/O1)
- D14 pad 3: D- DMCU-2 -> Net-(D14-I/O2)
- J7 pad A6: D+ DMCU-2 -> Net-(D14-I/O1)
- J7 pad A7: D- DMCU-2 -> Net-(D14-I/O2)
- J7 pad B6: D+ DMCU-2 -> Net-(D14-I/O1)
- J7 pad B7: D- DMCU-2 -> Net-(D14-I/O2)
- U5 pad 10: unconnected-(U5-PA05-Pad10) -> mosfet2_signalfire
- U5 pad 17: +3.3V -> GND
- U5 pad 36: +3.3V -> GND
- U5 pad 43: Net-(U5-VDDCORE) -> +3.3V
- U5 pad 44: +3.3V -> GND
- U5 pad 6: +3.3V -> GND
- U5 pad 9: unconnected-(U5-PA04-Pad9) -> mosfet1_signalfire
Routing:
- net GND: track 106.8 -> 93.1 mm, vias 127 -> 124
- net SWCLK DMCU-2: track 10.1 -> 22.6 mm
- net SWDIO DMCU-2: track 7.51 -> 16.6 mm, vias 0 -> 1
- net +3.3V: track 114.5 -> 117.2 mm, vias 8 -> 11
- net nRESET DMCU-2: track 11.6 -> 14.0 mm
- net Net-(U5-VDDCORE): track 2.01 -> 0.00 mm
- net (no net): track 0.00 -> 2.01 mm
Other:
- board size 34 x 34 mm -> 34 x 41.8 mm
